File: control_board/control_board.brd (EAGLE design)
At the start: 70 x 74.5 mm, 37 parts, among them IC1 ATMEGA1284P-MU, J1 USB Female Type C Connector, Q1 220mA/50V/3.5Ω, SW1 SPST_TACT-KMR2, U1 915MHz, U3 MCP73833

Commit message: updated control board (unfinished)
- Schematic complete
- all components placed on board in roughly the approx. location
Parts:
- removed C2: 1u, LowPowerLab:0603-CAP
- removed D2: GREEN, SparkFun-LED:LED-0603
- removed D3: Yellow, SparkFun-LED:LED-0603
- removed D4: (no value), adafruit:SOD-123
- removed Q1: 220mA/50V/3.5Ω, SparkFun-DiscreteSemi:SOT23-3
- added C10, C11, C12, C13, C6, C9: 0.1uF, Adafruit Feather 32u4 Bluefruit LE:MICROBUILDER__0402MP
- added C14: 10uF, Adafruit Feather 32u4 Bluefruit LE:MICROBUILDER__0402MP
- added C7: 10µF, SparkFun-Capacitors:0805
- added C8: 1uF, Adafruit Feather 32u4 Bluefruit LE:MICROBUILDER__0402MP
- added F1: 6V 0.5A, SparkFun-Fuses:0805
- added J3: (no value), SparkFun-Connectors:1X02
- added J4: (no value), SparkFun-Connectors:1X01
- added LED2: (no value), adafruit:CHIPLED_0603
- added Q2: BSS84-7-F, MOSFETs:SOT23-3
- added Q3: BSS138PW,115, MOSFETs:SOT323
- added R10, R9: 4.7K, Adafruit Feather 32u4 Bluefruit LE:MICROBUILDER__0402MP
- added R11, R12: 5.1K, Adafruit Feather 32u4 Bluefruit LE:MICROBUILDER__0402MP
- added R13, R14: 27, Adafruit Feather 32u4 Bluefruit LE:MICROBUILDER__0402MP
- added R16, R19, R20, R21, R22, R23, R8: 10K, Adafruit Feather 32u4 Bluefruit LE:MICROBUILDER__0402MP
- added R17, R18: 10M, Adafruit Feather 32u4 Bluefruit LE:MICROBUILDER__0402MP
- added R30: 330, Adafruit Feather 32u4 Bluefruit LE:MICROBUILDER__0402MP
- added U$8, U$9: FIDUCIAL, adafruit:FIDUCIAL_1MM
- C1: value 10uF -> 10µF; device SparkFun-Capacitors:0603 -> SparkFun-Capacitors:0805
- C3: value 10u -> 0.1uF; device LowPowerLab:0805-CAP -> Adafruit Feather 32u4 Bluefruit LE:MICROBUILDER__0402MP
- C4: value 0.1 -> 0.1uF; device LowPowerLab:0603-CAP -> Adafruit Feather 32u4 Bluefruit LE:MICROBUILDER__0402MP
- C5: device SparkFun-Capacitors:0603 -> Adafruit Feather 32u4 Bluefruit LE:MICROBUILDER__0402MP
- D1: value RED -> (none); device SparkFun-LED:LED-0603 -> SCHOTTKY_0805:0805
- LED1: device adafruit:CHIPLED_0805 -> adafruit:CHIPLED_0603
- R1: value 1.5k -> 330; device SparkFun-Resistors:0603 -> Adafruit Feather 32u4 Bluefruit LE:MICROBUILDER__0402MP
- R2: value 1.5k -> 10K; device SparkFun-Resistors:0603 -> Adafruit Feather 32u4 Bluefruit LE:MICROBUILDER__0402MP
- R3: value 1.5k -> 1K; device SparkFun-Resistors:0603 -> Adafruit Feather 32u4 Bluefruit LE:MICROBUILDER__0402MP
- R4: value 1k -> 100; device SparkFun-Resistors:0603 -> Adafruit Feather 32u4 Bluefruit LE:MICROBUILDER__0402MP
- R5: value PROG -> 10K; device SparkFun-Resistors:AXIAL-0.3 -> Adafruit Feather 32u4 Bluefruit LE:MICROBUILDER__0402MP
- R6: value 10k -> 330; device SparkFun-Resistors:0603 -> Adafruit Feather 32u4 Bluefruit LE:MICROBUILDER__0402MP
- R7: value THERM -> 330; device SparkFun-Resistors:AXIAL-0.3 -> Adafruit Feather 32u4 Bluefruit LE:MICROBUILDER__0402MP
- moved R7 36.1 mm to (32.9, 11.4)
- moved R5 33.9 mm to (36.7, 16.5)
- moved R4 31.2 mm to (9.90, 16.2)
- moved R2 21.6 mm to (22.1, 8.80)
- moved C3 20.8 mm to (28.5, 1.80)
- moved C4 17.9 mm to (24.6, 26.4)
- moved C1 17.2 mm to (21.7, 15.5), turned to 90 degrees
- moved D1 15.4 mm to (26.2, 9.90), turned to 90 degrees
- moved XTAL1 14.8 mm to (12.1, 25.8), turned to 90 degrees
- moved LED1 14.3 mm to (32.4, 16.2)
- moved R3 7.82 mm to (36.7, 18.4)
- moved R6 7.24 mm to (32.8, 13.2)
- moved U$1 5.39 mm to (27.1, 17.3)
- moved U3 4.95 mm to (38.7, 10.4)
- moved C5 4.70 mm to (36.8, 24.1), turned to 180 degrees
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Connections:
- removed net 3.3V: U1.13
- removed net AVCC: IC1.27
- removed net D11_MOSI: W25X40CLSNIG-ND.5_SI
- removed net D12_MISO: W25X40CLSNIG-ND.2_SO
- removed net D13_SCK: W25X40CLSNIG-ND.6_SCK
- removed net D8: W25X40CLSNIG-ND.1_CS
- removed net GND1: XTAL1.2
- removed net GND_1: IC1.18
- removed net GND_2: IC1.28
- removed net GND_3: IC1.39
- removed net N$21: XTAL1.3
- removed net PG: R3.2, U3.P$7
- removed net STAT1: R1.2, U3.P$3
- removed net STAT2: R2.2, U3.P$4
- removed net VCC_1: IC1.17
- removed net VCC_2: IC1.38
- removed net VDD: C1.1, D1.A, D2.A, D3.A, U2.5, U3.P$1, U3.P$2
- removed net VSS: U2.8, U2.THERMAL
- removed net V_BATT: C5.1, J2.2, U3.P$10, U3.P$9
- new net 12V_SENSE: IC1.37, U$6.5
- new net A: C11.2, IC1.11, MT1.A, R19.2, R21.1, R21.2
- new net ANT: J4.1, U1.9
- new net B: C13.2, IC1.12, MT1.B, R20.2, R22.1, R22.2
- new net CHARGE: R1.1, R30.1, U3.P$3
- new net CS: IC1.26, W25X40CLSNIG-ND.1_CS
- new net CURRENT_SENSE_POWER: IC1.24, U$4.10
- new net D2: IC1.42, U1.14
- new net DTR: U$1.DTR#
- new net FTDI_3.3V: Q3.1, R2.1, R6.1, R7.1, U$1.3V3OUT, U$1.RESET#, U$1.VCCIO
- new net IN1: IC1.13, U$4.1
- new net IN2: IC1.14, U$4.2
- new net KNOB: IC1.40, MT1.2
- new net MISO: IC1.2, TC1.1, U1.2, W25X40CLSNIG-ND.2_SO
- new net MOSI: IC1.1, TC1.4, U1.3, W25X40CLSNIG-ND.5_SI
- new net MOTOR_CONTROL: IC1.25, U$4.8
- new net N$10: F1.1, J1.VBUS1, J1.VBUS2
- new net N$11: MT1.1, R23.1
- new net N$12: R4.2, SW1.1, SW1.3
- new net N$13: LED1.C, U$1.CBUS2
- new net N$14: Q3.2, R2.2, U$1.RXD
- new net N$15: LED1.A, R6.2
- new net N$17: LED2.A, R7.2
- new net N$18: LED2.C, U$1.CBUS1
- new net N$2: C14.2, J2.2, J3.2, U3.P$10, U3.P$9
- new net N$3: IC1.7, XTAL1.3
- new net N$7: J1.A7, J1.B7, R13.2
- new net N$8: R14.1, U$1.USBDP
- new net N$9: R13.1, U$1.USBDM
- new net PWR: C5.2, TC1.2, U3.P$1, U3.P$2
- new net RESET: C12.2, IC1.4, R4.1, R8.2, TC1.5
- new net RX: IC1.9, U$1.TXD
- new net SCK: IC1.3, TC1.3, U1.4, W25X40CLSNIG-ND.6_SCK
- new net SS: IC1.44, U1.5
- new net TEMP: IC1.34, U$4.3
- new net TEMP_SENSOR_POWER: C10.1, IC1.23, U2.5
- new net TX: IC1.10, Q3.3
- new net VBAT: J3.1, Q2.3, R17.2, U$7.10, U$7.7, U$7.8, U$7.9
- new net VBAT_SENSE: C9.1, IC1.30, R17.1, R18.1
- new net VBUS: C3.1, D1.1, F1.2, Q2.1, R16.2, U$1.VCC
- net BLUE: now also IC1.16
- net GND: now also C10.2, C11.1, C12.1, C13.1, C14.1, C5.1, C6.2, C7.1, C8.2, C9.2, IC1.18, IC1.28, IC1.39, IC1.45, J1.GND, J1.GND2, MT1.COM, R11.2, R12.2, R16.1, R18.2, R23.2, R3.2, R5.2, SW1.2, SW1.4, TC1.6, U$1.GND_PIN13, U$1.GND_PIN21, U$1.GND_PIN3, U$4.5, U$4.6, U$6.7, U$6.8, U$7.1, U$7.2, U2.7, U2.8, U2.THERMAL, XTAL1.2; no longer C2.2, C5.2, R4.1, R5.P$1, R6.1, R7.P$1
- net GREEN: now also R1.2, U3.P$4
- net N$1: now also IC1.8
- net N$4: now also J1.B5, R11.1; no longer D1.C, R3.1
- net N$5: now also J1.A5, R12.1; no longer D2.C, R2.1
- net N$6: now also J1.A6, J1.B6, R14.2; no longer D3.C, R1.1
- net PROG: now also R3.1; no longer R4.2, R5.P$2
- net RED: now also R30.2
- net SCL: now also IC1.19, R10.1, U$6.10, U2.4
- net SDA: now also IC1.20, R9.1, U$6.9, U2.1
- net SDB: now also IC1.22
- net THERM: now also R5.1; no longer R6.2, R7.P$2
- net VCC: now also C1.1, C6.1, C7.2, IC1.17, IC1.27, IC1.38, R10.2, R19.1, R20.1, R8.1, R9.2, U$6.1, U$6.2, U1.13; no longer C3.1
- net VIN: now also C8.1, D1.2, Q2.2; no longer C2.1

Commit message: v0.1 - finished design
- Added gerbers, renders, dxf
- Updated dimensions
Parts:
- removed MCP1703: MCP1703CB, linear:SOT23
- removed U$6, U$7: 20021311-00010T4LF, Amphenol:HEADER_1.27MM_2X5
- added J5, J6: 20021311-00010T4LF, Amphenol:HEADER_1.27MM_2X5
- added U4: MCP1703CB, linear:SOT23
- F1: value 6V 0.5A -> 10V 1.5A
- moved C11 22.8 mm to (48.4, 33.4), turned to 270 degrees
- moved R22 20.7 mm to (45.3, 36.6), turned to 270 degrees
- moved R20 20.3 mm to (46.9, 36.6), turned to 90 degrees
- moved C13 19.5 mm to (48.4, 36.6), turned to 90 degrees
- moved R21 19.2 mm to (45.3, 33.4), turned to 90 degrees
- moved R19 17.3 mm to (46.9, 33.4), turned to 270 degrees
- moved C14 17.0 mm to (39.9, 9.40), turned to 90 degrees
- moved Q3 13.2 mm to (33.7, 12.0), turned to 270 degrees
- moved C7 13.1 mm to (7.70, 52.3), turned to 0 degrees
- moved R7 12.9 mm to (35.4, 24.0), turned to 180 degrees
- moved R2 9.90 mm to (31.5, 11.8), turned to 270 degrees
- moved C6 9.62 mm to (21.1, 13.3)
- moved R11 9.40 mm to (36.7, 6.10)
- moved R14 9.31 mm to (35.6, 6.10), turned to 270 degrees
- moved R6 9.28 mm to (35.4, 22.1), turned to 180 degrees
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- renumbered U$1 to U8, U$4 to J7, U$5 to U5, W25X40CLSNIG-ND to U7
Connections:
- net N$2 renamed VBAT_CHG
- removed net PWR: C5.2, TC1.2, U3.P$1, U3.P$2
- new net CHANNEL_A: IC1.11, R21.2
- new net CHANNEL_B: IC1.12, R22.2
- net 12V_SENSE: now also J6.5; no longer U$6.5
- net A: no longer IC1.11, R21.2
- net B: no longer IC1.12, R22.2
- net DTR: now also C12.1
- net GND: now also J5.1, J5.2, J6.7, J6.8, U4.1; no longer C12.1, MCP1703.1, U$6.7, U$6.8, U$7.1, U$7.2
- net SCL: now also J6.10; no longer U$6.10
- net SDA: now also J6.9; no longer U$6.9
- net VBAT: now also J5.10, J5.7, J5.8, J5.9; no longer U$7.10, U$7.7, U$7.8, U$7.9
- net VBUS: now also C5.2, TC1.2, U3.P$1, U3.P$2
- net VCC: now also J6.1, J6.2, U4.2; no longer MCP1703.2, U$6.1, U$6.2
- net VIN: now also U4.3; no longer MCP1703.3
Routing:
- net VCC: track 0.00 -> 175.3 mm, vias 0 -> 9
- net VBUS: track 0.00 -> 95.6 mm, vias 0 -> 5
- net SCL: track 0.00 -> 91.8 mm, vias 0 -> 4
- net SDA: track 0.00 -> 87.6 mm, vias 0 -> 4
- net GREEN: track 0.00 -> 72.6 mm, vias 0 -> 6
- net TEMP_SENSOR_POWER: track 0.00 -> 70.5 mm, vias 0 -> 2
- net MISO: track 0.00 -> 69.3 mm, vias 0 -> 5
- net SCK: track 0.00 -> 61.9 mm, vias 0 -> 6
- net RED: track 0.00 -> 59.7 mm, vias 0 -> 4
- net CURRENT_SENSE_POWER: track 0.00 -> 56.5 mm, vias 0 -> 2
- net TEMP: track 0.00 -> 56.2 mm, vias 0 -> 1
- net RX: track 0.00 -> 55.6 mm, vias 0 -> 2
- net MOSI: track 0.00 -> 55.3 mm, vias 0 -> 4
- net MOTOR_CONTROL: track 0.00 -> 53.8 mm, vias 0 -> 2
- net VBAT: track 0.00 -> 53.8 mm, vias 0 -> 1
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- added copper zone on layer 1, net GND
- added copper zone on layer 16, net GND
- added copper zone on layer 1, net VBAT_CHG
- added copper zone on layer 1, net VBUS
Other:
- board size 70 x 74.5 mm -> 63 x 73.3 mm
- board text added: "915 MHz antenna"
- board text added: "<- LED screen conn. (contacts face down)"
- board text added: "BORC"
- board text added: "Battery conn."
- board text added: "Control Board"
- board text added: "Designed by Akram Ali"
- board text added: "Reset"
- board text added: "Temp sensor ->"
- board text added: "on/off switch"
- board text added: "v0.1 2020-11-16"
