File: control_board/control_board.sch (EAGLE design)
At the start: 70 parts, among them IC1 ATMEGA1284P-MU, J1 USB Female Type C Connector, J5 20021311-00010T4LF, J6 20021311-00010T4LF, J7 20021311-00010T4LF, Q2 BSS84-7-F, Q3 BSS138PW,115, SW1 SPST_TACT-KMR2, U1 915MHz, U4 MCP1703CB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

Commit message: v0.7 - control board update
- Added pull up resistor to SHT31 ADDR pin (address changed from 0x44 to 0x45)
- Added cutout to control board to allow power board to be screwed from top
- Added cutout to FPC connector
- Rearranged some traces and components - slight adjustments
- gerbers updated
Parts:
- added R25: 10K, Adafruit Feather 32u4 Bluefruit LE:MICROBUILDER_RESISTOR_0402MP
- C1, C7: value 10µF -> 0.33µF
- F1: value 10V 1.5A -> 6V 0.5A
- J1: device SparkFun-Connectors:USB_C -> SparkFun-Connectors:USB_C_2-LAYER_PADS
Connections:
- new net N$20: R25.2, U2.ADDR
- net TEMP_SENSOR_POWER: now also R25.1
Changed lines of the file:
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@@
 </classes>
 <parts>
-<part name="IC1" library="ATMEGA1284P-MU" deviceset="ATMEGA1284P-MU" device="" override_package3d_urn="urn:adsk.eagle:package:24879864/2" override_package_urn="urn:adsk.eagle:footprint:24879865/1"/>
+<part name="IC1" library="ATMEGA1284P-MU" deviceset="ATMEGA1284P-MU" device="" override_package3d_urn="urn:adsk.eagle:package:24879864/2" override_package_urn="urn:adsk.eagle:footprint:24879865/1" override_locally_modified="yes"/>
 <part name="U1" library="SparkFun-RF" library_urn="urn:adsk.eagle:library:531" deviceset="RFM69H" device="CW-915" package3d_urn="urn:adsk.eagle:package:39566/1" override_package3d_urn="urn:adsk.eagle:package:24879983/2" override_package_urn="urn:adsk.eagle:footprint:39514/1" value="915MHz"/>
 <part name="SUPPLY8" library="supply2" library_urn="urn:adsk.eagle:library:372" deviceset="GND" device=""/>
@@
 <part name="U7" library="LowPowerLab" deviceset="AT25F512B" device="JEDEC_3.9MM" override_package3d_urn="urn:adsk.eagle:package:24877226/2" override_package_urn="urn:adsk.eagle:footprint:24877227/1" value="AT25F512BJEDEC_3.9MM"/>
 <part name="U8" library="ftdi_ft231xq-r" deviceset="FT231XQ-R" device="" override_package3d_urn="urn:adsk.eagle:package:24879808/2" override_package_urn="urn:adsk.eagle:footprint:24879809/1"/>
-<part name="J1" library="SparkFun-Connectors" deviceset="USB_C" device="" override_package3d_urn="urn:adsk.eagle:package:24877297/2" override_package_urn="urn:adsk.eagle:footprint:24877298/1" value="USB Female Type C Connector"/>
+<part name="J1" library="SparkFun-Connectors" deviceset="USB_C" device="_2-LAYER_PADS" override_package3d_urn="urn:adsk.eagle:package:24877297/2" override_package_urn="urn:adsk.eagle:footprint:24877298/1" override_locally_modified="yes" value="USB Female Type C Connector"/>
 <part name="SUPPLY3" library="SparkFun" deviceset="VCC" device="" value="3.3V"/>
 <part name="U4" library="linear" deviceset="MCP1703" device="CB" override_package3d_urn="urn:adsk.eagle:package:24879829/2" override_package_urn="urn:adsk.eagle:footprint:24879831/1"/>
@@
 <part name="GND9" library="SparkFun-PowerSymbols" deviceset="GND" device=""/>
 <part name="P+6" library="SparkFun" deviceset="VCC" device="" value="3.3V"/>
-<part name="F1" library="SparkFun-Fuses" deviceset="PPTC" device="_6V500MA" override_package3d_urn="urn:adsk.eagle:package:22384550/2" override_package_urn="urn:adsk.eagle:footprint:22384551/1" value="10V 1.5A">
+<part name="F1" library="SparkFun-Fuses" deviceset="PPTC" device="_6V500MA" override_package3d_urn="urn:adsk.eagle:package:22384550/2" override_package_urn="urn:adsk.eagle:footprint:22384551/1" value="6V 0.5A">
 <attribute name="MPN" value="MF-PSML110-2"/>
 </part>
@@
 </part>
 <part name="Q3" library="MOSFETs" deviceset="MOSFET-NCH" device="-BSS138PW,115" override_package3d_urn="urn:adsk.eagle:package:24877326/2" override_package_urn="urn:adsk.eagle:footprint:24877328/1" value="BSS138PW,115"/>
-<part name="LED1" library="adafruit" deviceset="LED" device="CHIPLED_0603" override_package3d_urn="urn:adsk.eagle:package:24879791/2" override_package_urn="urn:adsk.eagle:footprint:24879792/1"/>
-<part name="LED2" library="adafruit" deviceset="LED" device="CHIPLED_0603" override_package3d_urn="urn:adsk.eagle:package:24879794/2" override_package_urn="urn:adsk.eagle:footprint:24879795/1"/>
-<part name="C1" library="SparkFun-Capacitors" deviceset="0.33UF/330NF" device="-0805-50V-10%" override_package3d_urn="urn:adsk.eagle:package:24879823/2" override_package_urn="urn:adsk.eagle:footprint:24879824/1" value="10µF"/>
-<part name="C7" library="SparkFun-Capacitors" deviceset="0.33UF/330NF" device="-0805-50V-10%" override_package3d_urn="urn:adsk.eagle:package:24879912/2" override_package_urn="urn:adsk.eagle:footprint:24879913/1" value="10µF"/>
+<part name="LED1" library="adafruit" deviceset="LED" device="CHIPLED_0603" package3d_urn="urn:adsk.eagle:package:6240561/1" override_package3d_urn="urn:adsk.eagle:package:24879791/2" override_package_urn="urn:adsk.eagle:footprint:24879792/1" override_locally_modified="yes"/>
+<part name="LED2" library="adafruit" deviceset="LED" device="CHIPLED_0603" package3d_urn="urn:adsk.eagle:package:6240561/1" override_package3d_urn="urn:adsk.eagle:package:24879794/2" override_package_urn="urn:adsk.eagle:footprint:24879795/1" override_locally_modified="yes"/>
+<part name="C1" library="SparkFun-Capacitors" deviceset="0.33UF/330NF" device="-0805-50V-10%" override_package3d_urn="urn:adsk.eagle:package:24879823/2" override_package_urn="urn:adsk.eagle:footprint:24879824/1" override_locally_modified="yes" value="0.33µF"/>
+<part name="C7" library="SparkFun-Capacitors" deviceset="0.33UF/330NF" device="-0805-50V-10%" override_package3d_urn="urn:adsk.eagle:package:24879912/2" override_package_urn="urn:adsk.eagle:footprint:24879913/1" override_locally_modified="yes" value="0.33µF"/>
 <part name="R15" library="Adafruit Feather 32u4 Bluefruit LE" deviceset="MICROBUILDER_RESISTOR" device="_0402MP" override_package3d_urn="urn:adsk.eagle:package:24877243/2" override_package_urn="urn:adsk.eagle:footprint:24877244/1" value="10K">
 <attribute name="MPN" value="RC0402FR-7W10KL"/>
@@
 </part>
 <part name="P+8" library="SparkFun" deviceset="VCC" device="" value="3.3V"/>
-<part name="LED3" library="adafruit" deviceset="LED" device="CHIPLED_0603" override_package3d_urn="urn:adsk.eagle:package:24879794/2" override_package_urn="urn:adsk.eagle:footprint:24879795/1" value="PWR"/>
+<part name="LED3" library="adafruit" deviceset="LED" device="CHIPLED_0603" package3d_urn="urn:adsk.eagle:package:6240561/1" override_package3d_urn="urn:adsk.eagle:package:24879794/2" override_package_urn="urn:adsk.eagle:footprint:24879795/1" override_locally_modified="yes" value="PWR"/>
 <part name="R1" library="Adafruit Feather 32u4 Bluefruit LE" deviceset="MICROBUILDER_RESISTOR" device="_0402MP" override_package3d_urn="urn:adsk.eagle:package:24877291/2" override_package_urn="urn:adsk.eagle:footprint:24877292/1" value="1K">
 <attribute name="MPN" value="RC0402FR-7W10KL"/>
@@
 </part>
 <part name="GND25" library="supply1" library_urn="urn:adsk.eagle:library:371" deviceset="GND" device=""/>
+<part name="R25" library="Adafruit Feather 32u4 Bluefruit LE" deviceset="MICROBUILDER_RESISTOR" device="_0402MP" override_package3d_urn="urn:adsk.eagle:package:24877243/2" override_package_urn="urn:adsk.eagle:footprint:24877244/1" value="10K">
+<attribute name="MPN" value="RC0402FR-7W10KL"/>
+</part>
 </parts>
 <sheets>
@@
 </instance>
 <instance part="J1" gate="J1" x="0" y="-60.96" smashed="yes">
-<attribute name="VALUE" x="-5.334" y="-78.74" size="1.778" layer="96" font="vector" rot="MR90" align="top-left"/>
 <attribute name="NAME" x="-2.54" y="-50.546" size="1.778" layer="95" font="vector"/>
 </instance>
@@
 <instance part="GND25" gate="1" x="-50.8" y="134.62" smashed="yes">
 <attribute name="VALUE" x="-53.34" y="132.08" size="1.778" layer="96"/>
+</instance>
+<instance part="R25" gate="G$1" x="226.06" y="73.66" smashed="yes" rot="R270">
+<attribute name="MPN" x="226.06" y="73.66" size="1.778" layer="96" rot="R270" display="off"/>
+<attribute name="NAME" x="228.6" y="73.66" size="1.4224" layer="95" rot="R270" align="center"/>
+<attribute name="VALUE" x="223.52" y="73.66" size="1.4224" layer="96" ratio="15" rot="R270" align="center"/>
 </instance>
 </instances>
@@
 <segment>
 <pinref part="U2" gate="G$1" pin="VDD"/>
-<wire x1="256.54" y1="71.12" x2="269.24" y2="71.12" width="0.1524" layer="91"/>
+<wire x1="256.54" y1="71.12" x2="259.08" y2="71.12" width="0.1524" layer="91"/>
 <pinref part="C10" gate="G$1" pin="1"/>
 <label x="259.08" y="71.12" size="1.778" layer="95"/>
+<pinref part="R25" gate="G$1" pin="1"/>
+<wire x1="259.08" y1="71.12" x2="269.24" y2="71.12" width="0.1524" layer="91"/>
+<wire x1="226.06" y1="78.74" x2="226.06" y2="83.82" width="0.1524" layer="91"/>
+<wire x1="226.06" y1="83.82" x2="259.08" y2="83.82" width="0.1524" layer="91"/>
+<wire x1="259.08" y1="83.82" x2="259.08" y2="71.12" width="0.1524" layer="91"/>
+<junction x="259.08" y="71.12"/>
 </segment>
 </net>
@@
 </segment>
 </net>
+<net name="N$20" class="0">
+<segment>
+<pinref part="U2" gate="G$1" pin="ADDR"/>
+<pinref part="R25" gate="G$1" pin="2"/>
+<wire x1="231.14" y1="66.04" x2="226.06" y2="66.04" width="0.1524" layer="91"/>
+<wire x1="226.06" y1="66.04" x2="226.06" y2="68.58" width="0.1524" layer="91"/>
+</segment>
+</net>
