File: hardware/power_board/power_board.sch (EAGLE design)
At the start: 36 parts, among them J5 20021311-00010T4LF, J6 20021311-00010T4LF, J7 20021311-00010T4LF, Q1 600mA/40V, Q3 600mA/40V, Q4 NTMD4184PFR2G, U11 INA219AIDCNR, U5 POLOLU_STEPUP_U1V11X

Commit message: power board upgraded to v0.5
- added footprint for Pololu U3V40F5
- thickened several power traces even more
- added flyback diode to 5V line
- rearranged some traces to accommodate mods
- updated schematic, gerbers, render, dimensions
- ERC/DRC
Parts:
- added C7: 0.1uF, Adafruit Feather 32u4 Bluefruit LE:MICROBUILDER_CAP_CERAMIC_0402MP
- added D1: 1N4148, microbuilder:DIODESOD-323
- added U6: POLOLU_STEPUP_U3V40X, Pololu Step Up Vregs:POLOLU_STEPUP_U3V40X
Connections:
- net 5V: now also C7.1, D1.C, U6.VOUT
- net GND: now also C7.2, D1.A, U6.GND
- net VBAT_ON: now also U6.VIN
Other:
- moved on the sheet: R43
